File: PocketBeagle.sch (KiCad schematic (older format))
At the start: 28 parts, among them J1 Conn_01x08_Male, J10 Conn_01x04_Male, J11 Conn_01x04_Male, J12 Conn_01x04_Male, J13 Conn_01x04_Male, J14 Conn_01x04_Male, J15 Conn_01x04_Male, J16 Conn_01x04_Male, J17 Conn_01x02_Male, J18 Conn_01x02_Male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

Commit message: Correct misalignment and delete unnecessary files. 位置ずれの修正と、不要なファイルの削除。
Parts:
- removed J1, J4: Conn_01x08_Male, pocketbeagle:j vcc, symbol Connector:Conn_01x08_Male
- removed J10, J11, J12, J13, J14, J15, J16, J2, J21, J22, J27, J28, J3, J5, J6, J7, J8, J9: Conn_01x04_Male, pocketbeagle:yb, symbol Connector:Conn_01x04_Male
- removed J17, J18, J23, J24: Conn_01x02_Male, pocketbeagle:j 2, symbol Connector:Conn_01x02_Male
- removed J19, J20, J25, J26: Conn_01x01_Male, pocketbeagle:j 1, symbol Connector:Conn_01x01_Male
- added J1, J2, J3, J4: Conn_01x18_Male, Connector_PinHeader_2.54mm:PinHeader_1x18_P2.54mm_Vertical, symbol Connector:Conn_01x18_Male
- added J10, J11, J12, J13, J14, J15, J16, J17, J18, J19, J20, J21, J22, J23, J24, J7, J8, J9: Conn_01x08_Male, Connector_PinHeader_2.54mm:PinHeader_1x08_P2.54mm_Vertical, symbol Connector:Conn_01x08_Male
- added J5, J6: Conn_01x10_Male, Connector_PinHeader_2.54mm:PinHeader_1x10_P2.54mm_Vertical, symbol Connector:Conn_01x10_Male
Connections:
- wire segments 20 -> 0
